Commit message: updated spot with arm

File: spot_description/urdf/spot_with_arm.urdf (robot description, URDF)
Before this commit: robot spot_with_arm, 35 links, 34 joints
Links:
- removed link camera_depth_frame
- removed link camera_depth_optical_frame
- removed link camera_link
- removed link camera_rgb_frame
- removed link camera_rgb_optical_frame
- removed link hokuyo_frame
- added link frontleft_depth_frame
- added link frontleft_depth_optical_frame
- added link frontleft_link
- added link frontleft_rgb_frame
- added link frontleft_rgb_optical_frame
- added link frontright_depth_frame
- added link frontright_depth_optical_frame
- added link frontright_link
- added link frontright_rgb_frame
- added link frontright_rgb_optical_frame
- link body: mass 16.0 -> 32.0
Joints:
- removed joint camera_depth_joint
- removed joint camera_depth_optical_joint
- removed joint camera_joint
- removed joint camera_rgb_joint
- removed joint camera_rgb_optical_joint
- removed joint hokuyo_joint
- added joint frontleft: type fixed, parent base_link, child frontleft_link, origin xyz=0.405 0.035  -0.02 rpy=-1.8326 0.349066 -0.698132
- added joint frontleft_depth_joint: type fixed, parent frontleft_link, child frontleft_depth_frame, origin xyz=0.0 0.049 0.0 rpy=0 0 0
- added joint frontleft_depth_optical_joint: type fixed, parent frontleft_depth_frame, child frontleft_depth_optical_frame, origin xyz=0 0 0 rpy=-1.57079632679 0.0 -1.57079632679
- added joint frontleft_rgb_joint: type fixed, parent frontleft_link, child frontleft_rgb_frame, origin xyz=0.0 0.022 0.0 rpy=0 0 0
- added joint frontleft_rgb_optical_joint: type fixed, parent frontleft_rgb_frame, child frontleft_rgb_optical_frame, origin xyz=0 0 0 rpy=-1.57079632679 0.0 -1.57079632679
- added joint frontright: type fixed, parent base_link, child frontright_link, origin xyz=0.405 -0.035 -0.02 rpy=-1.309 0.349066 0.698132
- added joint frontright_depth_joint: type fixed, parent frontright_link, child frontright_depth_frame, origin xyz=0.0 0.049 0.0 rpy=0 0 0
- added joint frontright_depth_optical_joint: type fixed, parent frontright_depth_frame, child frontright_depth_optical_frame, origin xyz=0 0 0 rpy=-1.57079632679 0.0 -1.57079632679
- added joint frontright_rgb_joint: type fixed, parent frontright_link, child frontright_rgb_frame, origin xyz=0.0 0.022 0.0 rpy=0 0 0
- added joint frontright_rgb_optical_joint: type fixed, parent frontright_rgb_frame, child frontright_rgb_optical_frame, origin xyz=0 0 0 rpy=-1.57079632679 0.0 -1.57079632679

File: spot_description/urdf/spot_with_arm.xacro (robot description, xacro)
@@ -1,5 +1,5 @@
 <?xml version="1.0" encoding="utf-8"?>
 <robot xmlns:xacro="http://www.ros.org/wiki/xacro" name="spot_with_arm">
-  <xacro:include filename="$(find spot_description)/urdf/spot.urdf.xacro"/>
+  <xacro:include filename="$(find spot_description)/urdf/spot.urdf"/>
   <xacro:include filename="$(find spot_description)/urdf/spot_arm.xacro"/>
 <joint name="arm_mount" type="fixed">
