Commit message: changed cmaera dpeth range and robot mass

File: spot_description/urdf/spot.urdf (robot description, URDF)
Before this commit: robot spot, 31 links, 30 joints
Links:
- link body: mass 16.0 -> 32.0

Commit message: update urdfs

File: spot_description/urdf/spot.urdf (robot description, URDF)
Before this commit: robot spot, 31 links, 30 joints
Links:
- link body: mass 32.0 -> 20.0

File: spot_description/urdf/spot_with_arm.urdf (robot description, URDF)
Before this commit: robot spot_with_arm, 39 links, 38 joints
Links:
- link body: mass 32.0 -> 20.0
Joints:
- joint arm_mount: origin xyz=0 0 0 rpy=0 0 0 -> xyz=0 0 0 rpy=0 0 1.57079632679

File: spot_description/urdf/spot_with_arm.xacro (robot description, xacro)
@@ -4,5 +4,5 @@
   <xacro:include filename="$(find spot_description)/urdf/spot_arm.xacro"/>
 <joint name="arm_mount" type="fixed">
-      <origin xyz="0 0 0" rpy="0 0 0" />
+      <origin xyz="0 0 0" rpy="0 0 1.57079632679" />
       <parent link="front_rail" />
       <child link="base" />
