Commit message: update urdf mistake

File: spot_description/urdf/spot_arm.xacro (robot description, xacro)
@@ -13,5 +13,5 @@
     <origin rpy="0 0 0" xyz="0 0 0"/>
     <geometry>
-      <mesh filename="package://spot_arm_description/meshes/base_link.stl" scale="0.001 0.001 0.001"/>
+      <mesh filename="package://spot_description/meshes/base_link.stl" scale="0.001 0.001 0.001"/>
     </geometry>
     <material name="silver"/>
@@ -20,5 +20,5 @@
     <origin rpy="0 0 0" xyz="0 0 0"/>
     <geometry>
-      <mesh filename="package://spot_arm_description/meshes/base_link.stl" scale="0.001 0.001 0.001"/>
+      <mesh filename="package://spot_description/meshes/base_link.stl" scale="0.001 0.001 0.001"/>
     </geometry>
   </collision>
@@ -33,5 +33,5 @@
     <origin rpy="0 0 0" xyz="0.001 -0.4505 -0.0475"/>
     <geometry>
-      <mesh filename="package://spot_arm_description/meshes/Part3_1.stl" scale="0.001 0.001 0.001"/>
+      <mesh filename="package://spot_description/meshes/Part3_1.stl" scale="0.001 0.001 0.001"/>
     </geometry>
     <material name="silver"/>
@@ -40,5 +40,5 @@
     <origin rpy="0 0 0" xyz="0.001 -0.4505 -0.0475"/>
     <geometry>
-      <mesh filename="package://spot_arm_description/meshes/Part3_1.stl" scale="0.001 0.001 0.001"/>
+      <mesh filename="package://spot_description/meshes/Part3_1.stl" scale="0.001 0.001 0.001"/>
     </geometry>
   </collision>
@@ -53,5 +53,5 @@
     <origin rpy="0 0 0" xyz="0.0085 -0.77959 -0.0475"/>
     <geometry>
-      <mesh filename="package://spot_arm_description/meshes/gripper_1.stl" scale="0.001 0.001 0.001"/>
+      <mesh filename="package://spot_description/meshes/gripper_1.stl" scale="0.001 0.001 0.001"/>
     </geometry>
     <material name="silver"/>
@@ -60,5 +60,5 @@
     <origin rpy="0 0 0" xyz="0.0085 -0.77959 -0.0475"/>
     <geometry>
-      <mesh filename="package://spot_arm_description/meshes/gripper_1.stl" scale="0.001 0.001 0.001"/>
+      <mesh filename="package://spot_description/meshes/gripper_1.stl" scale="0.001 0.001 0.001"/>
     </geometry>
   </collision>
@@ -73,5 +73,5 @@
     <origin rpy="0 0 0" xyz="0.87709 -0.823505 -0.0185"/>
     <geometry>
-      <mesh filename="package://spot_arm_description/meshes/finger_1.stl" scale="0.001 0.001 0.001"/>
+      <mesh filename="package://spot_description/meshes/finger_1.stl" scale="0.001 0.001 0.001"/>
     </geometry>
     <material name="silver"/>
@@ -80,5 +80,5 @@
     <origin rpy="0 0 0" xyz="0.87709 -0.823505 -0.0185"/>
     <geometry>
-      <mesh filename="package://spot_arm_description/meshes/finger_1.stl" scale="0.001 0.001 0.001"/>
+      <mesh filename="package://spot_description/meshes/finger_1.stl" scale="0.001 0.001 0.001"/>
     </geometry>
   </collision>
@@ -93,5 +93,5 @@
     <origin rpy="0 0 0" xyz="-0.015 -0.0 -0.115"/>
     <geometry>
-      <mesh filename="package://spot_arm_description/meshes/Part1_1.stl" scale="0.001 0.001 0.001"/>
+      <mesh filename="package://spot_description/meshes/Part1_1.stl" scale="0.001 0.001 0.001"/>
     </geometry>
     <material name="silver"/>
@@ -100,5 +100,5 @@
     <origin rpy="0 0 0" xyz="-0.015 -0.0 -0.115"/>
     <geometry>
-      <mesh filename="package://spot_arm_description/meshes/Part1_1.stl" scale="0.001 0.001 0.001"/>
+      <mesh filename="package://spot_description/meshes/Part1_1.stl" scale="0.001 0.001 0.001"/>
     </geometry>
   </collision>
@@ -113,5 +113,5 @@
     <origin rpy="0 0 0" xyz="-0.0 -0.0 -0.065"/>
     <geometry>
-      <mesh filename="package://spot_arm_description/meshes/Part0_1.stl" scale="0.001 0.001 0.001"/>
+      <mesh filename="package://spot_description/meshes/Part0_1.stl" scale="0.001 0.001 0.001"/>
     </geometry>
     <material name="silver"/>
@@ -120,5 +120,5 @@
     <origin rpy="0 0 0" xyz="-0.0 -0.0 -0.065"/>
     <geometry>
-      <mesh filename="package://spot_arm_description/meshes/Part0_1.stl" scale="0.001 0.001 0.001"/>
+      <mesh filename="package://spot_description/meshes/Part0_1.stl" scale="0.001 0.001 0.001"/>
     </geometry>
   </collision>
@@ -133,5 +133,5 @@
     <origin rpy="0 0 0" xyz="0.0485 -0.69859 -0.0475"/>
     <geometry>
-      <mesh filename="package://spot_arm_description/meshes/Part4_1.stl" scale="0.001 0.001 0.001"/>
+      <mesh filename="package://spot_description/meshes/Part4_1.stl" scale="0.001 0.001 0.001"/>
     </geometry>
     <material name="silver"/>
@@ -140,5 +140,5 @@
     <origin rpy="0 0 0" xyz="0.0485 -0.69859 -0.0475"/>
     <geometry>
-      <mesh filename="package://spot_arm_description/meshes/Part4_1.stl" scale="0.001 0.001 0.001"/>
+      <mesh filename="package://spot_description/meshes/Part4_1.stl" scale="0.001 0.001 0.001"/>
     </geometry>
   </collision>
@@ -153,5 +153,5 @@
     <origin rpy="0 0 0" xyz="-0.017 -0.3125 -0.115"/>
     <geometry>
-      <mesh filename="package://spot_arm_description/meshes/Part2_1.stl" scale="0.001 0.001 0.001"/>
+      <mesh filename="package://spot_description/meshes/Part2_1.stl" scale="0.001 0.001 0.001"/>
     </geometry>
     <material name="silver"/>
@@ -160,5 +160,5 @@
     <origin rpy="0 0 0" xyz="-0.017 -0.3125 -0.115"/>
     <geometry>
-      <mesh filename="package://spot_arm_description/meshes/Part2_1.stl" scale="0.001 0.001 0.001"/>
+      <mesh filename="package://spot_description/meshes/Part2_1.stl" scale="0.001 0.001 0.001"/>
     </geometry>
   </collision>

File: spot_description/urdf/spot_with_arm.urdf (robot description, URDF)
Before this commit: robot spot_with_arm, 39 links, 38 joints
Links:
- link Part0_1: geometry collision mesh filename=package://spot_description/meshes/Part0_1.stl scale=0.001 0.001 0.001; visual mesh filename=package://spot_description/meshes/Part0_1.stl scale=0.001 0.001 0.001
- link Part1_1: geometry collision mesh filename=package://spot_description/meshes/Part1_1.stl scale=0.001 0.001 0.001; visual mesh filename=package://spot_description/meshes/Part1_1.stl scale=0.001 0.001 0.001
- link Part2_1: geometry collision mesh filename=package://spot_description/meshes/Part2_1.stl scale=0.001 0.001 0.001; visual mesh filename=package://spot_description/meshes/Part2_1.stl scale=0.001 0.001 0.001
- link Part3_1: geometry collision mesh filename=package://spot_description/meshes/Part3_1.stl scale=0.001 0.001 0.001; visual mesh filename=package://spot_description/meshes/Part3_1.stl scale=0.001 0.001 0.001
- link Part4_1: geometry collision mesh filename=package://spot_description/meshes/Part4_1.stl scale=0.001 0.001 0.001; visual mesh filename=package://spot_description/meshes/Part4_1.stl scale=0.001 0.001 0.001
- link base: geometry collision mesh filename=package://spot_description/meshes/base_link.stl scale=0.001 0.001 0.001; visual mesh filename=package://spot_description/meshes/base_link.stl scale=0.001 0.001 0.001
- link finger_1: geometry collision mesh filename=package://spot_description/meshes/finger_1.stl scale=0.001 0.001 0.001; visual mesh filename=package://spot_description/meshes/finger_1.stl scale=0.001 0.001 0.001
- link gripper_1: geometry collision mesh filename=package://spot_description/meshes/gripper_1.stl scale=0.001 0.001 0.001; visual mesh filename=package://spot_description/meshes/gripper_1.stl scale=0.001 0.001 0.001
